File: wejscia_analogowe_2.kicad_sch (KiCad schematic)
At the start: 30 parts

Commit message: Zaktualizowano pliki
Parts:
- R155, R156, R69, R70, R71, R77, R78, R79, R82, R87, R93, R96: Manufacturer TE Connectivity AMP -> Panasonic; Manufacturer Part Number RP73PF1E15KBTDF -> ERA-2VEB7501X
Changed lines of the file:
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@@
 			)
 		)
-		(property "Datasheet" "https://octopart.com/datasheet/te-connectivity-amp/2176312-9"
+		(property "Datasheet" "https://industrial.panasonic.com/cdbs/www-data/pdf/RDM0000/RDM0000C331.pdf"
 			(at 63.5 97.79 0)
 			(effects
@@
 			)
 		)
-		(property "Description" "15 kOhms ±0.1% 0.1W, 1/10W Chip Resistor 0402 (1005 Metric) Thin Film"
+		(property "Description" "7.5 kOhms ±0.1% 0.1W, 1/10W Chip Resistor 0402 (1005 Metric) Anti-Sulfur, Automotive AEC-Q200 Thin Film"
 			(at 63.5 97.79 0)
 			(effects
@@
 			)
 		)
-		(property "Manufacturer" "TE Connectivity AMP"
+		(property "Manufacturer" "Panasonic"
 			(at 63.5 97.79 0)
 			(effects
@@
 			)
 		)
-		(property "Manufacturer Part Number" "RP73PF1E15KBTDF"
+		(property "Manufacturer Part Number" "ERA-2VEB7501X"
 			(at 63.5 97.79 0)
 			(effects
@@
 			)
 		)
-		(property "Datasheet" "https://octopart.com/datasheet/te-connectivity-amp/2176312-9"
+		(property "Datasheet" "https://industrial.panasonic.com/cdbs/www-data/pdf/RDM0000/RDM0000C331.pdf"
 			(at 229.87 40.64 0)
 			(effects
@@
 			)
 		)
-		(property "Description" "15 kOhms ±0.1% 0.1W, 1/10W Chip Resistor 0402 (1005 Metric) Thin Film"
+		(property "Description" "7.5 kOhms ±0.1% 0.1W, 1/10W Chip Resistor 0402 (1005 Metric) Anti-Sulfur, Automotive AEC-Q200 Thin Film"
 			(at 229.87 40.64 0)
 			(effects
@@
 			)
 		)
-		(property "Manufacturer" "TE Connectivity AMP"
+		(property "Manufacturer" "Panasonic"
 			(at 229.87 40.64 0)
 			(effects
@@
 			)
 		)
-		(property "Manufacturer Part Number" "RP73PF1E15KBTDF"
+		(property "Manufacturer Part Number" "ERA-2VEB7501X"
 			(at 229.87 40.64 0)
 			(effects
@@
 			)
 		)
-		(property "Datasheet" "https://octopart.com/datasheet/te-connectivity-amp/2176312-9"
+		(property "Datasheet" "https://industrial.panasonic.com/cdbs/www-data/pdf/RDM0000/RDM0000C331.pdf"
 			(at 152.4 113.03 0)
 			(effects
@@
 			)
 		)
-		(property "Description" "15 kOhms ±0.1% 0.1W, 1/10W Chip Resistor 0402 (1005 Metric) Thin Film"
+		(property "Description" "7.5 kOhms ±0.1% 0.1W, 1/10W Chip Resistor 0402 (1005 Metric) Anti-Sulfur, Automotive AEC-Q200 Thin Film"
 			(at 152.4 113.03 0)
 			(effects
@@
 			)
 		)
-		(property "Manufacturer" "TE Connectivity AMP"
+		(property "Manufacturer" "Panasonic"
 			(at 152.4 113.03 0)
 			(effects
@@
 			)
 		)
-		(property "Manufacturer Part Number" "RP73PF1E15KBTDF"
+		(property "Manufacturer Part Number" "ERA-2VEB7501X"
 			(at 152.4 113.03 0)
 			(effects
@@
 			)
 		)
-		(property "Datasheet" "https://octopart.com/datasheet/te-connectivity-amp/2176312-9"
+		(property "Datasheet" "https://industrial.panasonic.com/cdbs/www-data/pdf/RDM0000/RDM0000C331.pdf"
 			(at 143.51 46.99 0)
 			(effects
@@
 			)
 		)
-		(property "Description" "15 kOhms ±0.1% 0.1W, 1/10W Chip Resistor 0402 (1005 Metric) Thin Film"
+		(property "Description" "7.5 kOhms ±0.1% 0.1W, 1/10W Chip Resistor 0402 (1005 Metric) Anti-Sulfur, Automotive AEC-Q200 Thin Film"
 			(at 143.51 46.99 0)
 			(effects
@@
 			)
 		)
-		(property "Manufacturer" "TE Connectivity AMP"
+		(property "Manufacturer" "Panasonic"
 			(at 143.51 46.99 0)
 			(effects
@@
 			)
 		)
-		(property "Manufacturer Part Number" "RP73PF1E15KBTDF"
+		(property "Manufacturer Part Number" "ERA-2VEB7501X"
 			(at 143.51 46.99 0)
 			(effects
@@
 			)
 		)
-		(property "Datasheet" "https://octopart.com/datasheet/te-connectivity-amp/2176312-9"
+		(property "Datasheet" "https://industrial.panasonic.com/cdbs/www-data/pdf/RDM0000/RDM0000C331.pdf"
 			(at 57.15 91.44 0)
 			(effects
@@
 			)
 		)
-		(property "Description" "15 kOhms ±0.1% 0.1W, 1/10W Chip Resistor 0402 (1005 Metric) Thin Film"
+		(property "Description" "7.5 kOhms ±0.1% 0.1W, 1/10W Chip Resistor 0402 (1005 Metric) Anti-Sulfur, Automotive AEC-Q200 Thin Film"
 			(at 57.15 91.44 0)
 			(effects
@@
 			)
 		)
-		(property "Manufacturer" "TE Connectivity AMP"
+		(property "Manufacturer" "Panasonic"
 			(at 57.15 91.44 0)
 			(effects
@@
 			)
 		)
-		(property "Manufacturer Part Number" "RP73PF1E15KBTDF"
+		(property "Manufacturer Part Number" "ERA-2VEB7501X"
 			(at 57.15 91.44 0)
 			(effects
@@
 			)
 		)
-		(property "Datasheet" "https://octopart.com/datasheet/te-connectivity-amp/2176312-9"
+		(property "Datasheet" "https://industrial.panasonic.com/cdbs/www-data/pdf/RDM0000/RDM0000C331.pdf"
 			(at 231.14 90.17 0)
 			(effects
@@
 			)
 		)
-		(property "Description" "15 kOhms ±0.1% 0.1W, 1/10W Chip Resistor 0402 (1005 Metric) Thin Film"
+		(property "Description" "7.5 kOhms ±0.1% 0.1W, 1/10W Chip Resistor 0402 (1005 Metric) Anti-Sulfur, Automotive AEC-Q200 Thin Film"
 			(at 231.14 90.17 0)
 			(effects
@@
 			)
 		)
-		(property "Manufacturer" "TE Connectivity AMP"
+		(property "Manufacturer" "Panasonic"
 			(at 231.14 90.17 0)
 			(effects
@@
 			)
 		)
-		(property "Manufacturer Part Number" "RP73PF1E15KBTDF"
+		(property "Manufacturer Part Number" "ERA-2VEB7501X"
 			(at 231.14 90.17 0)
 			(effects
@@
 			)
 		)
-		(property "Datasheet" "https://octopart.com/datasheet/te-connectivity-amp/2176312-9"
+		(property "Datasheet" "https://industrial.panasonic.com/cdbs/www-data/pdf/RDM0000/RDM0000C331.pdf"
 			(at 137.16 40.64 0)
 			(effects
@@
 			)
 		)
-		(property "Description" "15 kOhms ±0.1% 0.1W, 1/10W Chip Resistor 0402 (1005 Metric) Thin Film"
+		(property "Description" "7.5 kOhms ±0.1% 0.1W, 1/10W Chip Resistor 0402 (1005 Metric) Anti-Sulfur, Automotive AEC-Q200 Thin Film"
 			(at 137.16 40.64 0)
 			(effects
@@
 			)
 		)
-		(property "Manufacturer" "TE Connectivity AMP"
+		(property "Manufacturer" "Panasonic"
 			(at 137.16 40.64 0)
 			(effects
@@
 			)
 		)
-		(property "Manufacturer Part Number" "RP73PF1E15KBTDF"
+		(property "Manufacturer Part Number" "ERA-2VEB7501X"
 			(at 137.16 40.64 0)
 			(effects
@@
 			)
 		)
-		(property "Datasheet" "https://octopart.com/datasheet/te-connectivity-amp/2176312-9"
+		(property "Datasheet" "https://industrial.panasonic.com/cdbs/www-data/pdf/RDM0000/RDM0000C331.pdf"
 			(at 146.05 106.68 0)
 			(effects
@@
 			)
 		)
-		(property "Description" "15 kOhms ±0.1% 0.1W, 1/10W Chip Resistor 0402 (1005 Metric) Thin Film"
+		(property "Description" "7.5 kOhms ±0.1% 0.1W, 1/10W Chip Resistor 0402 (1005 Metric) Anti-Sulfur, Automotive AEC-Q200 Thin Film"
 			(at 146.05 106.68 0)
 			(effects
@@
 			)
 		)
-		(property "Manufacturer" "TE Connectivity AMP"
+		(property "Manufacturer" "Panasonic"
 			(at 146.05 106.68 0)
 			(effects
@@
 			)
 		)
-		(property "Manufacturer Part Number" "RP73PF1E15KBTDF"
+		(property "Manufacturer Part Number" "ERA-2VEB7501X"
 			(at 146.05 106.68 0)
 			(effects
@@
 			)
 		)
-		(property "Datasheet" "https://octopart.com/datasheet/te-connectivity-amp/2176312-9"
+		(property "Datasheet" "https://industrial.panasonic.com/cdbs/www-data/pdf/RDM0000/RDM0000C331.pdf"
 			(at 237.49 96.52 0)
 			(effects
@@
 			)
 		)
-		(property "Description" "15 kOhms ±0.1% 0.1W, 1/10W Chip Resistor 0402 (1005 Metric) Thin Film"
+		(property "Description" "7.5 kOhms ±0.1% 0.1W, 1/10W Chip Resistor 0402 (1005 Metric) Anti-Sulfur, Automotive AEC-Q200 Thin Film"
 			(at 237.49 96.52 0)
 			(effects
@@
 			)
 		)
-		(property "Manufacturer" "TE Connectivity AMP"
+		(property "Manufacturer" "Panasonic"
 			(at 237.49 96.52 0)
 			(effects
@@
 			)
 		)
-		(property "Manufacturer Part Number" "RP73PF1E15KBTDF"
+		(property "Manufacturer Part Number" "ERA-2VEB7501X"
 			(at 237.49 96.52 0)
 			(effects
@@
 			)
 		)
-		(property "Datasheet" "https://octopart.com/datasheet/te-connectivity-amp/2176312-9"
+		(property "Datasheet" "https://industrial.panasonic.com/cdbs/www-data/pdf/RDM0000/RDM0000C331.pdf"
 			(at 53.34 40.64 0)
 			(effects
@@
 			)
 		)
-		(property "Description" "15 kOhms ±0.1% 0.1W, 1/10W Chip Resistor 0402 (1005 Metric) Thin Film"
+		(property "Description" "7.5 kOhms ±0.1% 0.1W, 1/10W Chip Resistor 0402 (1005 Metric) Anti-Sulfur, Automotive AEC-Q200 Thin Film"
 			(at 53.34 40.64 0)
 			(effects
@@
 			)
 		)
-		(property "Manufacturer" "TE Connectivity AMP"
+		(property "Manufacturer" "Panasonic"
 			(at 53.34 40.64 0)
 			(effects
@@
 			)
 		)
-		(property "Manufacturer Part Number" "RP73PF1E15KBTDF"
+		(property "Manufacturer Part Number" "ERA-2VEB7501X"
 			(at 53.34 40.64 0)
 			(effects
@@
 			)
 		)
-		(property "Datasheet" "https://octopart.com/datasheet/te-connectivity-amp/2176312-9"
+		(property "Datasheet" "https://industrial.panasonic.com/cdbs/www-data/pdf/RDM0000/RDM0000C331.pdf"
 			(at 59.69 48.26 0)
 			(effects
@@
 			)
 		)
-		(property "Description" "15 kOhms ±0.1% 0.1W, 1/10W Chip Resistor 0402 (1005 Metric) Thin Film"
+		(property "Description" "7.5 kOhms ±0.1% 0.1W, 1/10W Chip Resistor 0402 (1005 Metric) Anti-Sulfur, Automotive AEC-Q200 Thin Film"
 			(at 59.69 48.26 0)
 			(effects
@@
 			)
 		)
-		(property "Manufacturer" "TE Connectivity AMP"
+		(property "Manufacturer" "Panasonic"
 			(at 59.69 48.26 0)
 			(effects
@@
 			)
 		)
-		(property "Manufacturer Part Number" "RP73PF1E15KBTDF"
+		(property "Manufacturer Part Number" "ERA-2VEB7501X"
 			(at 59.69 48.26 0)
 			(effects
@@
 			)
 		)
-		(property "Datasheet" "https://octopart.com/datasheet/te-connectivity-amp/2176312-9"
+		(property "Datasheet" "https://industrial.panasonic.com/cdbs/www-data/pdf/RDM0000/RDM0000C331.pdf"
 			(at 236.22 46.99 0)
 			(effects
@@
 			)
 		)
-		(property "Description" "15 kOhms ±0.1% 0.1W, 1/10W Chip Resistor 0402 (1005 Metric) Thin Film"
+		(property "Description" "7.5 kOhms ±0.1% 0.1W, 1/10W Chip Resistor 0402 (1005 Metric) Anti-Sulfur, Automotive AEC-Q200 Thin Film"
 			(at 236.22 46.99 0)
 			(effects
@@
 			)
 		)
-		(property "Manufacturer" "TE Connectivity AMP"
+		(property "Manufacturer" "Panasonic"
 			(at 236.22 46.99 0)
 			(effects
@@
 			)
 		)
-		(property "Manufacturer Part Number" "RP73PF1E15KBTDF"
+		(property "Manufacturer Part Number" "ERA-2VEB7501X"
 			(at 236.22 46.99 0)
 			(effects
