File: wejscia_analogowe_3.kicad_sch (KiCad schematic)
At the start: 25 parts

Commit message: Zaktualizowano pliki
Parts:
- R134, R135, R14, R143, R144, R148, R150, R152, R153, R91: Manufacturer TE Connectivity AMP -> Panasonic; Manufacturer Part Number RP73PF1E15KBTDF -> ERA-2VEB7501X
Changed lines of the file:
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@@
 			)
 		)
-		(property "Datasheet" "https://octopart.com/datasheet/te-connectivity-amp/2176312-9"
+		(property "Datasheet" "https://industrial.panasonic.com/cdbs/www-data/pdf/RDM0000/RDM0000C331.pdf"
 			(at 113.03 133.35 0)
 			(effects
@@
 			)
 		)
-		(property "Description" "15 kOhms ±0.1% 0.1W, 1/10W Chip Resistor 0402 (1005 Metric) Thin Film"
+		(property "Description" "7.5 kOhms ±0.1% 0.1W, 1/10W Chip Resistor 0402 (1005 Metric) Anti-Sulfur, Automotive AEC-Q200 Thin Film"
 			(at 113.03 133.35 0)
 			(effects
@@
 			)
 		)
-		(property "Manufacturer" "TE Connectivity AMP"
+		(property "Manufacturer" "Panasonic"
 			(at 113.03 133.35 0)
 			(effects
@@
 			)
 		)
-		(property "Manufacturer Part Number" "RP73PF1E15KBTDF"
+		(property "Manufacturer Part Number" "ERA-2VEB7501X"
 			(at 113.03 133.35 0)
 			(effects
@@
 			)
 		)
-		(property "Datasheet" "https://octopart.com/datasheet/te-connectivity-amp/2176312-9"
+		(property "Datasheet" "https://industrial.panasonic.com/cdbs/www-data/pdf/RDM0000/RDM0000C331.pdf"
 			(at 57.15 91.44 0)
 			(effects
@@
 			)
 		)
-		(property "Description" "15 kOhms ±0.1% 0.1W, 1/10W Chip Resistor 0402 (1005 Metric) Thin Film"
+		(property "Description" "7.5 kOhms ±0.1% 0.1W, 1/10W Chip Resistor 0402 (1005 Metric) Anti-Sulfur, Automotive AEC-Q200 Thin Film"
 			(at 57.15 91.44 0)
 			(effects
@@
 			)
 		)
-		(property "Manufacturer" "TE Connectivity AMP"
+		(property "Manufacturer" "Panasonic"
 			(at 57.15 91.44 0)
 			(effects
@@
 			)
 		)
-		(property "Manufacturer Part Number" "RP73PF1E15KBTDF"
+		(property "Manufacturer Part Number" "ERA-2VEB7501X"
 			(at 57.15 91.44 0)
 			(effects
@@
 			)
 		)
-		(property "Datasheet" "https://octopart.com/datasheet/te-connectivity-amp/2176312-9"
+		(property "Datasheet" "https://industrial.panasonic.com/cdbs/www-data/pdf/RDM0000/RDM0000C331.pdf"
 			(at 53.34 39.37 0)
 			(effects
@@
 			)
 		)
-		(property "Description" "15 kOhms ±0.1% 0.1W, 1/10W Chip Resistor 0402 (1005 Metric) Thin Film"
+		(property "Description" "7.5 kOhms ±0.1% 0.1W, 1/10W Chip Resistor 0402 (1005 Metric) Anti-Sulfur, Automotive AEC-Q200 Thin Film"
 			(at 53.34 39.37 0)
 			(effects
@@
 			)
 		)
-		(property "Manufacturer" "TE Connectivity AMP"
+		(property "Manufacturer" "Panasonic"
 			(at 53.34 39.37 0)
 			(effects
@@
 			)
 		)
-		(property "Manufacturer Part Number" "RP73PF1E15KBTDF"
+		(property "Manufacturer Part Number" "ERA-2VEB7501X"
 			(at 53.34 39.37 0)
 			(effects
@@
 			)
 		)
-		(property "Datasheet" "https://octopart.com/datasheet/te-connectivity-amp/2176312-9"
+		(property "Datasheet" "https://industrial.panasonic.com/cdbs/www-data/pdf/RDM0000/RDM0000C331.pdf"
 			(at 179.07 90.17 0)
 			(effects
@@
 			)
 		)
-		(property "Description" "15 kOhms ±0.1% 0.1W, 1/10W Chip Resistor 0402 (1005 Metric) Thin Film"
+		(property "Description" "7.5 kOhms ±0.1% 0.1W, 1/10W Chip Resistor 0402 (1005 Metric) Anti-Sulfur, Automotive AEC-Q200 Thin Film"
 			(at 179.07 90.17 0)
 			(effects
@@
 			)
 		)
-		(property "Manufacturer" "TE Connectivity AMP"
+		(property "Manufacturer" "Panasonic"
 			(at 179.07 90.17 0)
 			(effects
@@
 			)
 		)
-		(property "Manufacturer Part Number" "RP73PF1E15KBTDF"
+		(property "Manufacturer Part Number" "ERA-2VEB7501X"
 			(at 179.07 90.17 0)
 			(effects
@@
 			)
 		)
-		(property "Datasheet" "https://octopart.com/datasheet/te-connectivity-amp/2176312-9"
+		(property "Datasheet" "https://industrial.panasonic.com/cdbs/www-data/pdf/RDM0000/RDM0000C331.pdf"
 			(at 59.69 46.99 0)
 			(effects
@@
 			)
 		)
-		(property "Description" "15 kOhms ±0.1% 0.1W, 1/10W Chip Resistor 0402 (1005 Metric) Thin Film"
+		(property "Description" "7.5 kOhms ±0.1% 0.1W, 1/10W Chip Resistor 0402 (1005 Metric) Anti-Sulfur, Automotive AEC-Q200 Thin Film"
 			(at 59.69 46.99 0)
 			(effects
@@
 			)
 		)
-		(property "Manufacturer" "TE Connectivity AMP"
+		(property "Manufacturer" "Panasonic"
 			(at 59.69 46.99 0)
 			(effects
@@
 			)
 		)
-		(property "Manufacturer Part Number" "RP73PF1E15KBTDF"
+		(property "Manufacturer Part Number" "ERA-2VEB7501X"
 			(at 59.69 46.99 0)
 			(effects
@@
 			)
 		)
-		(property "Datasheet" "https://octopart.com/datasheet/te-connectivity-amp/2176312-9"
+		(property "Datasheet" "https://industrial.panasonic.com/cdbs/www-data/pdf/RDM0000/RDM0000C331.pdf"
 			(at 156.21 39.37 0)
 			(effects
@@
 			)
 		)
-		(property "Description" "15 kOhms ±0.1% 0.1W, 1/10W Chip Resistor 0402 (1005 Metric) Thin Film"
+		(property "Description" "7.5 kOhms ±0.1% 0.1W, 1/10W Chip Resistor 0402 (1005 Metric) Anti-Sulfur, Automotive AEC-Q200 Thin Film"
 			(at 156.21 39.37 0)
 			(effects
@@
 			)
 		)
-		(property "Manufacturer" "TE Connectivity AMP"
+		(property "Manufacturer" "Panasonic"
 			(at 156.21 39.37 0)
 			(effects
@@
 			)
 		)
-		(property "Manufacturer Part Number" "RP73PF1E15KBTDF"
+		(property "Manufacturer Part Number" "ERA-2VEB7501X"
 			(at 156.21 39.37 0)
 			(effects
@@
 			)
 		)
-		(property "Datasheet" "https://octopart.com/datasheet/te-connectivity-amp/2176312-9"
+		(property "Datasheet" "https://industrial.panasonic.com/cdbs/www-data/pdf/RDM0000/RDM0000C331.pdf"
 			(at 185.42 96.52 0)
 			(effects
@@
 			)
 		)
-		(property "Description" "15 kOhms ±0.1% 0.1W, 1/10W Chip Resistor 0402 (1005 Metric) Thin Film"
+		(property "Description" "7.5 kOhms ±0.1% 0.1W, 1/10W Chip Resistor 0402 (1005 Metric) Anti-Sulfur, Automotive AEC-Q200 Thin Film"
 			(at 185.42 96.52 0)
 			(effects
@@
 			)
 		)
-		(property "Manufacturer" "TE Connectivity AMP"
+		(property "Manufacturer" "Panasonic"
 			(at 185.42 96.52 0)
 			(effects
@@
 			)
 		)
-		(property "Manufacturer Part Number" "RP73PF1E15KBTDF"
+		(property "Manufacturer Part Number" "ERA-2VEB7501X"
 			(at 185.42 96.52 0)
 			(effects
@@
 			)
 		)
-		(property "Datasheet" "https://octopart.com/datasheet/te-connectivity-amp/2176312-9"
+		(property "Datasheet" "https://industrial.panasonic.com/cdbs/www-data/pdf/RDM0000/RDM0000C331.pdf"
 			(at 63.5 97.79 0)
 			(effects
@@
 			)
 		)
-		(property "Description" "15 kOhms ±0.1% 0.1W, 1/10W Chip Resistor 0402 (1005 Metric) Thin Film"
+		(property "Description" "7.5 kOhms ±0.1% 0.1W, 1/10W Chip Resistor 0402 (1005 Metric) Anti-Sulfur, Automotive AEC-Q200 Thin Film"
 			(at 63.5 97.79 0)
 			(effects
@@
 			)
 		)
-		(property "Manufacturer" "TE Connectivity AMP"
+		(property "Manufacturer" "Panasonic"
 			(at 63.5 97.79 0)
 			(effects
@@
 			)
 		)
-		(property "Manufacturer Part Number" "RP73PF1E15KBTDF"
+		(property "Manufacturer Part Number" "ERA-2VEB7501X"
 			(at 63.5 97.79 0)
 			(effects
@@
 			)
 		)
-		(property "Datasheet" "https://octopart.com/datasheet/te-connectivity-amp/2176312-9"
+		(property "Datasheet" "https://industrial.panasonic.com/cdbs/www-data/pdf/RDM0000/RDM0000C331.pdf"
 			(at 119.38 139.7 0)
 			(effects
@@
 			)
 		)
-		(property "Description" "15 kOhms ±0.1% 0.1W, 1/10W Chip Resistor 0402 (1005 Metric) Thin Film"
+		(property "Description" "7.5 kOhms ±0.1% 0.1W, 1/10W Chip Resistor 0402 (1005 Metric) Anti-Sulfur, Automotive AEC-Q200 Thin Film"
 			(at 119.38 139.7 0)
 			(effects
@@
 			)
 		)
-		(property "Manufacturer" "TE Connectivity AMP"
+		(property "Manufacturer" "Panasonic"
 			(at 119.38 139.7 0)
 			(effects
@@
 			)
 		)
-		(property "Manufacturer Part Number" "RP73PF1E15KBTDF"
+		(property "Manufacturer Part Number" "ERA-2VEB7501X"
 			(at 119.38 139.7 0)
 			(effects
@@
 			)
 		)
-		(property "Datasheet" "https://octopart.com/datasheet/te-connectivity-amp/2176312-9"
+		(property "Datasheet" "https://industrial.panasonic.com/cdbs/www-data/pdf/RDM0000/RDM0000C331.pdf"
 			(at 162.56 45.72 0)
 			(effects
@@
 			)
 		)
-		(property "Description" "15 kOhms ±0.1% 0.1W, 1/10W Chip Resistor 0402 (1005 Metric) Thin Film"
+		(property "Description" "7.5 kOhms ±0.1% 0.1W, 1/10W Chip Resistor 0402 (1005 Metric) Anti-Sulfur, Automotive AEC-Q200 Thin Film"
 			(at 162.56 45.72 0)
 			(effects
@@
 			)
 		)
-		(property "Manufacturer" "TE Connectivity AMP"
+		(property "Manufacturer" "Panasonic"
 			(at 162.56 45.72 0)
 			(effects
@@
 			)
 		)
-		(property "Manufacturer Part Number" "RP73PF1E15KBTDF"
+		(property "Manufacturer Part Number" "ERA-2VEB7501X"
 			(at 162.56 45.72 0)
 			(effects
