File: G473_dev_board.kicad_pcb (KiCad board)
At the start: 4 copper layers, 148 x 96 mm, 425 parts, among them J1 8-1241434-1, J2 Conn_01x04_Pin, J3 Conn_01x04_Pin, J4 Conn_01x02_Pin, J5 Conn_01x02_Pin, Q1 MMBTA06, Q10 MMFTP3401, Q11 2N7002H, Q12 MMFTP3401, Q13 2N7002H, Q14 MMFTP3401, Q15 MMBTA06, Q2 BC807, Q3 MMFTP3401, Q4 2N7002H, Q5 2N7002H, Q6 MMFTP3401, Q7 2N7002H, Q8 MMFTP3401, Q9 2N7002H, SW1 SW_Push, SW2 SW_Push, U1 STM32G473VETx, U10 74LVC1G17, U11 74LVC1G17, U12 74LVC1G17, U13 OPA333xxDBV, U15 74LVC1G17, U17 24LC512-E/SN, U18 OPA333xxDBV, U2 SIC438B, U3 TCAN330GD, U4 TCAN330GD, U5 TCAN330GD, U6 XC6220B331MR, U7 LM4030-2.5, U8 OPA333xxDBV, U9 74LVC1G17, Y1 ECS-3225MVLC-080-CN-TR, Y2 ECS-327ATQMV-AS-TR

Commit message: Zaktualizowano pliki
Parts:
- removed R127: 16.5k, Resistor_SMD:R_0402_1005Metric
- added C2: 0.1u, Capacitor_SMD:C_0402_1005Metric, F.Cu at (218.2, 147.9)
- added R160: 10k, Resistor_SMD:R_0402_1005Metric, F.Cu at (227.3, 144.8)
- added R90: 15k, Resistor_SMD:R_0402_1005Metric, F.Cu at (222.4, 142.6)
- added U14: OPA2333xxD, Package_SO:SOIC-8_3.9x4.9mm_P1.27mm, F.Cu at (222.9, 146.0)
- R115: value 5.1k -> 2.2k
- R116: value 100m -> 10R
- R34: value 100m -> 100R
- moved C72 0.20 mm to (229.0, 133.6)
- moved D14 0.10 mm to (230.2, 137.6)
- moved R122 0.10 mm to (230.2, 133.6), turned to 90 degrees
- turned R123 to 90 degrees
Connections:
- C72 pad 2: HVIL_SEND -> Net-(U14A-+)
- C74 pad 2: HVIL_RETURN -> Net-(U14B-+)
- D14 pad 3: HVIL_SEND -> HVIL_START
- D31 pad 3: HVIL_RETURN -> HVIL_END
- R122 pad 2: HVIL_SEND -> Net-(U14A-+)
- R123 pad 2: HVIL_RETURN -> Net-(U14B-+)
Routing:
- net Net-(U14A-+): track 0.00 -> 15.8 mm
- net Net-(U14B-+): track 0.00 -> 14.9 mm
- net HVIL_RETURN: track 69.0 -> 55.0 mm
- net HVIL_SEND: track 58.4 -> 47.4 mm
- net +5V: track 65.8 -> 70.7 mm, vias 14 -> 15
- net GND: track 518.4 -> 522.9 mm, vias 168 -> 171
- net HVIL_START: track 76.4 -> 79.4 mm
- net HVIL_END: track 113.9 -> 116.9 mm

Commit message: Zaktualizowano pliki
Parts:
- moved R80 0.10 mm to (166.8, 113.2)
Routing:
- net GND: track 522.9 -> 540.4 mm, vias 171 -> 167
- net PC10: track 98.6 -> 95.8 mm
- net PC11: track 140.3 -> 137.5 mm
- net PC2: track 148.4 -> 146.3 mm
- net PD2: track 151.4 -> 149.5 mm
- net +3V3: track 212.4 -> 214.2 mm
- net CAN3_RX: track 28.3 -> 30.1 mm
- net PD15: track 28.4 -> 26.9 mm
- net PD3: track 137.7 -> 136.2 mm
- net SPEED_SENS_5: track 90.6 -> 92.1 mm
- net PD11: track 50.5 -> 49.1 mm
- net PB12: track 68.2 -> 66.8 mm
- net PC3: track 149.0 -> 150.3 mm
- net PB4: track 19.2 -> 20.5 mm
- net PC1: track 144.2 -> 145.3 mm
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
Commit message: Zaktualizowano pliki
Parts:
- moved R43 8.66 mm to (181.3, 146.1), turned to -90 degrees
- moved R92 7.24 mm to (167.9, 139.2), turned to -90 degrees
- moved C1 5.90 mm to (166.1, 139.7)
- moved C76 5.28 mm to (165.6, 133.7)
- moved Y1 5.12 mm to (165.9, 131.3)
- moved R168 5.02 mm to (199.6, 127.1)
- moved R166 4.30 mm to (163.4, 130.8)
- moved U7 3.62 mm to (185.5, 146.2), turned to 180 degrees
- moved BT1 3.53 mm to (152.8, 121.5)
- moved C6 3.18 mm to (160.4, 126.8)
- moved R169 3.13 mm to (199.1, 129.2), turned to 0 degrees
- moved C5 3.04 mm to (184.3, 142.1), turned to 0 degrees
- moved R167 3.03 mm to (166.8, 126.0), turned to -90 degrees
- moved R85 2.81 mm to (181.1, 143.1)
- moved C4 2.80 mm to (181.6, 141.5)
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Connections:
- R170 pad 2: PB6 -> PF1
- U1 pad 13: GND -> PF1
- U1 pad 93: PB6 -> GND
- U10 pad 4: PD15 -> PC7
- U15 pad 4: PC7 -> PD15
Routing:
- net +3V3: track 214.2 -> 247.1 mm, vias 56 -> 60
- net PB6: track 32.5 -> 0.00 mm, vias 2 -> 0
- net PF1: track 0.00 -> 25.2 mm
- net GND: track 540.4 -> 558.9 mm, vias 167 -> 150
- net +5V: track 71.0 -> 85.6 mm, vias 15 -> 16
- net PD4: track 146.6 -> 159.3 mm
- net PD15: track 26.9 -> 15.7 mm, vias 2 -> 0
- net PC7: track 13.3 -> 24.5 mm
- net PD3: track 136.2 -> 145.9 mm
- net PD7: track 136.3 -> 145.1 mm
- net Net-(D15-K): track 7.69 -> 16.1 mm, vias 2 -> 4
- net PD5: track 137.8 -> 145.6 mm
- net PE10: track 131.7 -> 124.3 mm
- net VBAT: track 38.0 -> 45.2 mm
- net PD2: track 149.5 -> 156.6 mm
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