File: hso.kicad_sch (KiCad schematic)
At the start: 36 parts, among them Q10 MMFTP3401, Q3 MMFTP3401, Q4 2N7002H, Q5 2N7002H, Q6 MMFTP3401, Q7 2N7002H, Q8 MMFTP3401, Q9 2N7002H

Commit message: Zaktualizowano pliki
Changed lines of the file:
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@@
-		)
-	)
-	(global_label "PE2"
-		(shape input)
-		(at 119.38 77.47 0)
-		(fields_autoplaced yes)
-		(effects
-			(font
-				(size 1.27 1.27)
-			)
-			(justify left)
-		)
-		(property "Intersheetrefs" "${INTERSHEET_REFS}"
-			(at 125.9937 77.47 0)
-			(effects
-				(font
-					(size 1.27 1.27)
-				)
-				(justify left)
-				(hide yes)
-			)
 		)
 	)
