File: wejscia_cyfrowe_1.kicad_sch (KiCad schematic)
At the start: 35 parts, among them U15 74LVC1G17, U9 74LVC1G17

Commit message: Zaktualizowano pliki
Connections:
- net PC7 renamed PD15
Changed lines of the file:
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@@
 		)
 	)
-	(global_label "PC7"
+	(global_label "PD15"
 		(shape input)
 		(at 102.87 146.05 0)
@@
 		)
 		(property "Intersheetrefs" "${INTERSHEET_REFS}"
-			(at 109.6047 146.05 0)
+			(at 110.8142 146.05 0)
 			(effects
 				(font
