File: wejscia_cyfrowe_2.kicad_sch (KiCad schematic)
At the start: 40 parts, among them U10 74LVC1G17, U11 74LVC1G17, U12 74LVC1G17

Commit message: Zaktualizowano pliki
Connections:
- net PD15 renamed PC7
Changed lines of the file:
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@@
+		)
+	)
+	(global_label "PC7"
+		(shape input)
+		(at 167.64 50.8 0)
+		(fields_autoplaced yes)
+		(effects
+			(font
+				(size 1.27 1.27)
+			)
+			(justify left)
+		)
+		(property "Intersheetrefs" "${INTERSHEET_REFS}"
+			(at 174.3747 50.8 0)
+			(effects
+				(font
+					(size 1.27 1.27)
+				)
+				(justify left)
+				(hide yes)
+			)
 		)
 	)
@@
 			(effects
 				(font
-					(size 1.27 1.27)
-				)
-				(justify left)
-				(hide yes)
-			)
-		)
-	)
-	(global_label "PD15"
-		(shape input)
-		(at 167.64 50.8 0)
-		(fields_autoplaced yes)
-		(effects
-			(font
-				(size 1.27 1.27)
-			)
-			(justify left)
-		)
-		(property "Intersheetrefs" "${INTERSHEET_REFS}"
-			(at 175.5842 50.8 0)
-			(effects
-				(font
